File: hardware/servoboard/main.sch (KiCad schematic (older format))
At the start: 42 parts, among them IC1 ATMEGA8-P, K1 CS1, K10 CPOW2, K2 CS2, K3 CS3, K4 CS4, K5 CS5, K6 CS6, K7 CS7, K8 CS8, K9 CPOW, P1 PROG, P2 I2C, P3 JSE, Q1 IRFZ24N, X1 12MHz

Commit message: routing angefangen bugs fixed
Parts:
- removed P2: I2C, symbol CONN_2
- removed X1: 12MHz, symbol QUARTZCMS4
- added K11: I2C, symbol CONN_3
- added X1: 12MHz, symbol CRYSTAL
Connections:
- net GND: now also K11.3 (P3); no longer C11.2, C12.2, C13.2, C14.2, C6.2, C7.2, C8.2, C9.2
- net LED1: now also IC1.4 ((INT0)PD2); no longer IC1.2 ((RXD)PD0)
- net LED2: now also IC1.5 ((INT1)PD3); no longer IC1.3 ((TXD)PD1)
- net LED3: now also IC1.6 ((XCK/T0)PD4); no longer IC1.4 ((INT0)PD2)
- net S7: now also IC1.2 ((RXD)PD0); no longer IC1.27 ((ADC4/SDA)PC4)
- net S8: now also IC1.3 ((TXD)PD1); no longer IC1.28 ((ADC5/SCL)PC5)
- net SCL: now also IC1.28 ((ADC5/SCL)PC5), K11.2 (PM)
- net SDA: now also IC1.27 ((ADC4/SDA)PC4), K11.1 (P1)
- net SDrain: now also C11.2, C12.2, C13.2, C14.2, C6.2, C7.2, C8.2, C9.2, K1.3 (P3), K2.3 (P3), K3.3 (P3), K4.3 (P3), K5.3 (P3), K6.3 (P3), K7.3 (P3), K8.3 (P3)
- net SOnOff: no longer K1.3 (P3), K2.3 (P3), K3.3 (P3), K4.3 (P3), K5.3 (P3), K6.3 (P3), K7.3 (P3), K8.3 (P3)
- net at C2.2, IC1.10 (PB7(XTAL2/TOSC2)): now also X1.1
- net at C1.2, IC1.9 (PB6(XTAL1/TOSC1)): now also X1.2
