File: hardware/powerboard/main.kicad_pcb (KiCad board)
At the start: 2 copper layers, 34 parts, among them K1 jmp_servo, K2 jmp_laser, K3 jmp_12batt, P1 4-8V in, P10 servoL, P11 encoder, P12 servo_pow, P13 Laser, P14 FPGA, P15 12V reserve, P16 5v reserve, P17 usb_hub, P18 raspi, P19 servoL, P2 5V_in, P20 encoder, P21 servo_pow, P22 Laser, P23 FPGA, P24 12V reserve, P25 switch, P26 12V or Batt, P27 12V or Batt, P3 12V_in, P4 4-8V in, P5 5V_in, P6 12V_in, P7 5v reserve, P8 usb_hub, P9 raspi

Commit message: midterm presentation
Parts:
- moved D1 227.3 mm to (104.9, 69.9)
- moved D2 227.3 mm to (104.9, 77.9)
- moved K1 227.3 mm to (109.9, 63.9)
- moved K2 227.3 mm to (87.9, 63.9)
- moved K3 227.3 mm to (98.9, 63.9)
- moved P1 227.3 mm to (56.9, 62.9)
- moved P10 227.3 mm to (109.9, 94.9)
- moved P11 227.3 mm to (87.9, 94.9)
- moved P12 227.3 mm to (109.9, 52.9)
- moved P13 227.3 mm to (87.9, 52.9)
- moved P14 227.3 mm to (76.9, 52.9)
- moved P15 227.3 mm to (65.9, 52.9)
- moved P16 227.3 mm to (65.9, 87.9)
- moved P17 227.3 mm to (98.9, 87.9)
- moved P18 227.3 mm to (76.9, 87.9)
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